Commit message: Add files via upload

File: xacro/pendulum.xacro (robot description, xacro)
@@ -15,5 +15,5 @@
       <child  link="${prefix}_link"/>
       <axis xyz="0 0 1" />
-      <limit velocity="24.0" effort="0.4" />
+      <limit velocity="100.0" effort="0.4" />
       <dynamics damping="0.1"/>
     </joint>
@@ -47,6 +47,6 @@
     <gazebo reference="${prefix}_link">
       <material>Gazebo/Gray</material>
-      <mu1 value="2.5" />
-      <mu2 value="2.5" />
+      <mu1 value="1" />
+      <mu2 value="1" />
       <kp value="50000" />
       <kd value="10" />
@@ -84,5 +84,5 @@
   <xacro:wheel_macro prefix="left_wheel"  parent="base_link" xyz="0 0.11 0.05"/>
   <xacro:wheel_macro prefix="right_wheel" parent="base_link" xyz="0 -0.11 0.05"/>
-  <xacro:imu_macro prefix="imu" parent="base_link" xyz="0 0 0.20" robot_name="$(arg robot_name)"/>
+  <xacro:imu_macro prefix="imu" parent="base_link" xyz="0 0 0.50" robot_name="$(arg robot_name)"/>
   <gazebo>
     <plugin name="gazebo_ros_control" filename="libgazebo_ros_control.so">
